Commit message: adjust wheel

File: src/articubot_one/description/gazebo_control.xacro (robot description, xacro)
@@ -8,6 +8,6 @@
             <left_joint>back_left_wheel_joint</left_joint>
             <right_joint>back_right_wheel_joint</right_joint>
-            <wheel_separation>0.5</wheel_separation>  <!-- Distance between wheels (update if needed) -->
-            <wheel_diameter>0.1</wheel_diameter>        <!-- Diameter of the wheels (update if needed) -->
+            <wheel_separation>0.45</wheel_separation>  <!-- Distance between wheels (update if needed) -->
+            <wheel_diameter>0.14</wheel_diameter>        <!-- Diameter of the wheels (update if needed) -->
             <!-- Limits -->
             <max_wheel_torque>200</max_wheel_torque>
@@ -16,4 +16,5 @@
             <odometry_frame>odom</odometry_frame>
             <robot_base_frame>base_link</robot_base_frame>
+            <command_topic>diff_cont/cmd_vel_unstamped</command_topic>  <!-- Match twist_mux -->
             <publish_odom>true</publish_odom>
             <publish_odom_tf>true</publish_odom_tf>
@@ -24,6 +25,6 @@
             <left_joint>front_left_wheel_joint</left_joint>
             <right_joint>front_right_wheel_joint</right_joint>
-            <wheel_separation>0.5</wheel_separation>
-            <wheel_diameter>0.1</wheel_diameter>
+            <wheel_separation>0.45</wheel_separation>
+            <wheel_diameter>0.14</wheel_diameter>
             <!-- Limits -->
             <max_wheel_torque>200</max_wheel_torque>
@@ -32,4 +33,5 @@
             <odometry_frame>odom</odometry_frame>
             <robot_base_frame>base_link</robot_base_frame>
+            <command_topic>diff_cont/cmd_vel_unstamped</command_topic>  <!-- Match twist_mux -->
             <publish_odom>true</publish_odom>
             <publish_odom_tf>true</publish_odom_tf>

File: src/articubot_one/description/robot_core.xacro (robot description, xacro)
@@ -84,8 +84,8 @@
         <collision>
             <geometry>
-                <cylinder length="0.07" radius="0.05" />
-            </geometry>
-        </collision>
-        <xacro:inertial_cylinder mass="0.2" length="0.07" radius="0.07">
+                <cylinder length="0.075" radius="0.05" />
+            </geometry>
+        </collision>
+        <xacro:inertial_cylinder mass="0.2" length="0.075" radius="0.07">
             <origin xyz="0 0 0" rpy="0 0 0"/>
         </xacro:inertial_cylinder>
@@ -93,6 +93,6 @@
     <gazebo reference="front_left_wheel">
         <material>Gazebo/Blue</material>
-        <mu1 value="0.5"/>
-        <mu2 value="0.5"/>
+        <mu1 value="0.8"/>
+        <mu2 value="0.8"/>
     </gazebo>
     <!-- ==================================================  FRONT RIGHT WHEEL joint, link ================================================== -->
@@ -107,14 +107,14 @@
         <visual>
             <geometry>
+                <cylinder length="0.075" radius="0.07" />
+            </geometry>
+            <material name="blue"/>
+        </visual>
+        <collision>
+            <geometry>
                 <cylinder length="0.07" radius="0.07" />
             </geometry>
-            <material name="blue"/>
-        </visual>
-        <collision>
-            <geometry>
-                <cylinder length="0.07" radius="0.07" />
-            </geometry>
-        </collision>
-        <xacro:inertial_cylinder mass="0.2" length="0.07" radius="0.07">
+        </collision>
+        <xacro:inertial_cylinder mass="0.2" length="0.075" radius="0.07">
             <origin xyz="0 0 0" rpy="0 0 0"/>
         </xacro:inertial_cylinder>
@@ -122,64 +122,122 @@
     <gazebo reference="front_right_wheel">
         <material>Gazebo/Blue</material>
+        <mu1 value="0.8"/>
+        <mu2 value="0.8"/>
+    </gazebo>
+    <!-- ==================================================  BACK LEFT WHEEL joint, link ================================================== -->
+    <joint name="back_left_wheel_joint" type="continuous">
+        <parent link="base_link"/>
+        <child link="back_left_wheel"/>
+        <origin xyz="-0.09 0.225 0" rpy="-${pi/2} 0 0"/>
+        <axis xyz="0 0 1"/>
+    </joint>
+    <!-- ================================================== -->
+    <link name="back_left_wheel">
+        <visual>
+            <geometry>
+                <cylinder length="0.075" radius="0.07" />
+            </geometry>
+            <material name="gray"/>
+        </visual>
+        <collision>
+            <geometry>
+                <cylinder length="0.075" radius="0.07" />
+            </geometry>
+        </collision>
+        <xacro:inertial_cylinder mass="0.2" length="0.075" radius="0.07">
+            <origin xyz="0 0 0" rpy="0 0 0"/>
+        </xacro:inertial_cylinder>
+    </link>
+    <gazebo reference="back_left_wheel">
+        <material>Gazebo/Gray</material>
         <mu1 value="0.5"/>
         <mu2 value="0.5"/>
     </gazebo>
-    <!-- ==================================================  BACK LEFT WHEEL joint, link ================================================== -->
-    <joint name="back_left_wheel_joint" type="continuous">
-        <parent link="base_link"/>
-        <child link="back_left_wheel"/>
-        <origin xyz="-0.1 0.225 0" rpy="-${pi/2} 0 0"/>
-        <axis xyz="0 0 1"/>
-    </joint>
-    <!-- ================================================== -->
-    <link name="back_left_wheel">
-        <visual>
-            <geometry>
-                <cylinder length="0.07" radius="0.07" />
-            </geometry>
-            <material name="gray"/>
-        </visual>
-        <collision>
-            <geometry>
-                <cylinder length="0.07" radius="0.07" />
-            </geometry>
-        </collision>
-        <xacro:inertial_cylinder mass="0.2" length="0.07" radius="0.07">
-            <origin xyz="0 0 0" rpy="0 0 0"/>
-        </xacro:inertial_cylinder>
-    </link>
-    <gazebo reference="back_left_wheel">
+    <!-- ================================================== BACK RIGHT WHEEL joint, link ================================================== -->
+    <joint name="back_right_wheel_joint" type="continuous">
+        <parent link="base_link"/>
+        <child link="back_right_wheel"/>
+        <origin xyz="-0.09 -0.225 0" rpy="${pi/2} 0 0"/>
+        <axis xyz="0 0 -1"/>
+    </joint>
+    <!-- ================================================== -->
+    <link name="back_right_wheel">
+        <visual>
+            <geometry>
+                <cylinder length="0.075" radius="0.07" />
+            </geometry>
+            <material name="gray"/>
+        </visual>
+        <collision>
+            <geometry>
+                <cylinder length="0.075" radius="0.07" />
+            </geometry>
+        </collision>
+        <xacro:inertial_cylinder mass="0.2" length="0.075" radius="0.07">
+            <origin xyz="0 0 0" rpy="0 0 0"/>
+        </xacro:inertial_cylinder>
+    </link>
+    <gazebo reference="back_right_wheel">
         <material>Gazebo/Gray</material>
         <mu1 value="0.5"/>
         <mu2 value="0.5"/>
     </gazebo>
-    <!-- ================================================== BACK RIGHT WHEEL joint, link ================================================== -->
-    <joint name="back_right_wheel_joint" type="continuous">
-        <parent link="base_link"/>
-        <child link="back_right_wheel"/>
-        <origin xyz="-0.1 -0.225 0" rpy="${pi/2} 0 0"/>
-        <axis xyz="0 0 -1"/>
-    </joint>
-    <!-- ================================================== -->
-    <link name="back_right_wheel">
-        <visual>
-            <geometry>
-                <cylinder length="0.07" radius="0.07" />
-            </geometry>
-            <material name="gray"/>
-        </visual>
-        <collision>
-            <geometry>
-                <cylinder length="0.07" radius="0.07" />
-            </geometry>
-        </collision>
-        <xacro:inertial_cylinder mass="0.2" length="0.07" radius="0.07">
-            <origin xyz="0 0 0" rpy="0 0 0"/>
-        </xacro:inertial_cylinder>
-    </link>
-    <gazebo reference="back_right_wheel">
-        <material>Gazebo/Gray</material>
-        <mu1 value="0.5"/>
-        <mu2 value="0.5"/>
+    <!-- ================================================== REAR BACK LEFT WHEEL joint, link ================================================== -->
+    <joint name="rear_back_left_wheel_joint" type="fixed">
+        <parent link="base_link"/>
+        <child link="rear_back_left_wheel"/>
+        <origin xyz="-0.26 0.225 0.01" rpy="-${pi/2} 0 0"/>
+        <!--axis xyz="0 0 1"/-->
+    </joint>
+    <!-- ================================================== -->
+    <link name="rear_back_left_wheel">
+        <visual>
+            <geometry>
+                <cylinder length="0.07" radius="0.06" />
+            </geometry>
+            <material name="gray"/>
+        </visual>
+        <collision>
+            <geometry>
+                <cylinder length="0.07" radius="0.06" />
+            </geometry>
+        </collision>
+        <xacro:inertial_cylinder mass="0.2" length="0.07" radius="0.06">
+            <origin xyz="0 0 0" rpy="0 0 0"/>
+        </xacro:inertial_cylinder>
+    </link>
+    <gazebo reference="rear_back_left_wheel">
+        <material>Gazebo/Gray</material>
+        <mu1 value="0.3"/>
+        <mu2 value="0.3"/>
+    </gazebo>
+    <!-- ================================================== REAR BACK RIGHT WHEEL joint, link ================================================== -->
+    <joint name="rear_back_right_wheel_joint" type="fixed">
+        <parent link="base_link"/>
+        <child link="rear_back_right_wheel"/>
+        <origin xyz="-0.26 -0.225 0.01" rpy="${pi/2} 0 0"/>
+        <!--axis xyz="0 0 -1"/-->
+    </joint>
+    <!-- ================================================== -->
+    <link name="rear_back_right_wheel">
+        <visual>
+            <geometry>
+                <cylinder length="0.07" radius="0.06" />
+            </geometry>
+            <material name="gray"/>
+        </visual>
+        <collision>
+            <geometry>
+                <cylinder length="0.07" radius="0.06" />
+            </geometry>
+        </collision>
+        <xacro:inertial_cylinder mass="0.2" length="0.07" radius="0.06">
+            <origin xyz="0 0 0" rpy="0 0 0"/>
+        </xacro:inertial_cylinder>
+    </link>
+    <gazebo reference="rear_back_right_wheel">
+        <material>Gazebo/Gray</material>
+        <mu1 value="0.3"/>
+        <mu2 value="0.3"/>
     </gazebo>
 </robot>

Commit message: fix diff drive

File: src/articubot_one/description/gazebo_control.xacro (robot description, xacro)
@@ -6,11 +6,14 @@
             <!-- <left_joint>front_left_wheel_joint</left_joint> -->
             <!-- <right_joint>front_right_wheel_joint</right_joint> -->
+            <num_wheel_pairs>2</num_wheel_pairs>
             <left_joint>back_left_wheel_joint</left_joint>
             <right_joint>back_right_wheel_joint</right_joint>
+            <left_joint>front_left_wheel_joint</left_joint>
+            <right_joint>front_right_wheel_joint</right_joint>
             <wheel_separation>0.45</wheel_separation>  <!-- Distance between wheels (update if needed) -->
             <wheel_diameter>0.14</wheel_diameter>        <!-- Diameter of the wheels (update if needed) -->
             <!-- Limits -->
-            <max_wheel_torque>200</max_wheel_torque>
-            <max_wheel_acceleration>10.0</max_wheel_acceleration>
+            <max_wheel_torque>300</max_wheel_torque>
+            <max_wheel_acceleration>15.0</max_wheel_acceleration>
             <!-- Output -->
             <odometry_frame>odom</odometry_frame>
@@ -21,13 +24,13 @@
             <publish_wheel_tf>true</publish_wheel_tf>
         </plugin>
-        <plugin name='front_wheel' filename='libgazebo_ros_diff_drive.so'>
+        <plugin name='rear_wheel' filename='libgazebo_ros_diff_drive.so'>
             <!-- Wheel Information -->
-            <left_joint>front_left_wheel_joint</left_joint>
-            <right_joint>front_right_wheel_joint</right_joint>
+            <left_joint>rear_back_left_wheel_joint</left_joint>
+            <right_joint>rear_back_right_wheel_joint</right_joint>
             <wheel_separation>0.45</wheel_separation>
             <wheel_diameter>0.14</wheel_diameter>
             <!-- Limits -->
-            <max_wheel_torque>200</max_wheel_torque>
-            <max_wheel_acceleration>10.0</max_wheel_acceleration>
+            <max_wheel_torque>300</max_wheel_torque>
+            <max_wheel_acceleration>15.0</max_wheel_acceleration>
             <!-- Output -->
             <odometry_frame>odom</odometry_frame>

File: src/articubot_one/description/robot_core.xacro (robot description, xacro)
@@ -25,4 +25,7 @@
         <color rgba="1 0.4 0.7 1" />
     </material>
+    <material name="cyan" >
+    <color rgba="0.0 1.0 1.0 1.0" />
+  </material>
     <!-- BASE LINK -->
     <link name="base_link">
@@ -46,7 +49,7 @@
     <link name="chassis">
         <visual>
-            <origin xyz="0 0 0.1" rpy="0 0 0"/>
-            <geometry>
-                <box size="0.7 0.5 0.15"/>
+            <origin xyz="-0.05 0 0.1" rpy="0 0 0"/>
+            <geometry>
+                <box size="0.6 0.5 0.15"/>
             </geometry>
             <material name="white"/>
@@ -55,8 +58,8 @@
             <origin xyz="0 0 0.075" rpy="0 0 0"/>
             <geometry>
-                <box size="0.7 0.5 0.15"/>
-            </geometry>
-        </collision>
-        <xacro:inertial_box mass="0.8" x="0.7" y="0.5" z="0.15">
+                <box size="0.6 0.5 0.15"/>
+            </geometry>
+        </collision>
+        <xacro:inertial_box mass="0.4" x="0.6" y="0.5" z="0.15">
             <origin xyz="0 0 0.075" rpy="0 0 0"/>
         </xacro:inertial_box>
@@ -66,4 +69,90 @@
         <mu1 value="0.5"/>
         <mu2 value="0.5"/>
+    </gazebo>
+    <!-- ================================================== LEFT BUMPER (Rounded Edge) ================================================== -->
+    <joint name="left_bumper_joint" type="fixed">
+        <parent link="chassis"/>
+        <child link="left_bumper"/>
+        <origin xyz="0.247 0.2 0.09" rpy="0 0 0"/>  <!-- Front edge of chassis -->
+    </joint>
+    <!-- ================================================== -->
+    <link name="left_bumper">
+        <visual>
+            <geometry>
+                <cylinder length="0.12" radius="0.05"/>  <!-- Half chassis height -->
+            </geometry>
+            <material name="white"/>
+        </visual>
+        <collision>
+            <geometry>
+                <cylinder length="0.12" radius="0.05"/>
+            </geometry>
+        </collision>
+        <xacro:inertial_cylinder mass="0.1" length="0.12" radius="0.05">
+            <origin xyz="0 0 0" rpy="0 0 0"/>
+        </xacro:inertial_cylinder>
+    </link>
+    <gazebo reference="left_bumper">
+        <material>Gazebo/White</material>
+        <mu1 value="0.3"/>  <!-- Smoother sliding -->
+        <mu2 value="0.3"/>
+    </gazebo>
+    <!-- ================================================== RIGHT BUMPER (Rounded Edge) ================================================== -->
+    <joint name="right_bumper_joint" type="fixed">
+        <parent link="chassis"/>
+        <child link="right_bumper"/>
+        <origin xyz="0.247 -0.2 0.09" rpy="0 0 0"/>  <!-- Rear edge of chassis -->
+    </joint>
+    <!-- ================================================== -->
+    <link name="right_bumper">
+        <visual>
+            <geometry>
+                <cylinder length="0.12" radius="0.05"/>
+            </geometry>
+            <material name="white"/>
+        </visual>
+        <collision>
+            <geometry>
+                <cylinder length="0.12" radius="0.05"/>
+            </geometry>
+        </collision>
+        <xacro:inertial_cylinder mass="0.1" length="0.12" radius="0.05">
+            <origin xyz="0 0 0" rpy="0 0 0"/>
+        </xacro:inertial_cylinder>
+    </link>
+    <gazebo reference="right_bumper">
+        <material>Gazebo/White</material>
+        <mu1 value="0.3"/>
+        <mu2 value="0.3"/>
+    </gazebo>
+    <!-- ==================================================  FRONT BUMPER joint, link ================================================== -->
+    <joint name="front_bumper_joint" type="fixed">
+        <parent link="base_link"/>
+        <child link="front_bumper"/>
+        <origin xyz="0 0 0"/>
+    </joint>
+    <!-- ================================================== -->
+    <link name="front_bumper">
+        <visual>
+            <origin xyz="0.273 0 0.09" rpy="0 0 0"/>
+            <geometry>
+                <box size="0.05 0.4 0.1"/>
+            </geometry>
+            <material name="blue"/>
+        </visual>
+        <collision>
+            <origin xyz="0 0 0.05" rpy="0 0 0"/>
+            <geometry>
+                <box size="0.05 0.4 0.1"/>
+            </geometry>
+        </collision>
+        <xacro:inertial_box mass="0.1" x="0.05" y="0.4" z="0.1">
+            <origin xyz="0 0 0.05" rpy="0 0 0"/>
+        </xacro:inertial_box>
+    </link>
+    <gazebo reference="front_bumper">
+        <material>Gazebo/Blue</material>
+        <mu1 value="0.3"/>
+        <mu2 value="0.3"/>
     </gazebo>
     <!-- ==================================================  FRONT LEFT WHEEL joint, link ================================================== -->
@@ -184,9 +273,9 @@
     </gazebo>
     <!-- ================================================== REAR BACK LEFT WHEEL joint, link ================================================== -->
-    <joint name="rear_back_left_wheel_joint" type="fixed">
+    <joint name="rear_back_left_wheel_joint" type="continuous">
         <parent link="base_link"/>
         <child link="rear_back_left_wheel"/>
-        <origin xyz="-0.26 0.225 0.01" rpy="-${pi/2} 0 0"/>
-        <!--axis xyz="0 0 1"/-->
+        <origin xyz="-0.26 0.225 0" rpy="-${pi/2} 0 0"/>
+        <axis xyz="0 0 1"/>
     </joint>
     <!-- ================================================== -->
@@ -194,5 +283,5 @@
         <visual>
             <geometry>
-                <cylinder length="0.07" radius="0.06" />
+                <cylinder length="0.075" radius="0.07" />
             </geometry>
             <material name="gray"/>
@@ -200,8 +289,8 @@
         <collision>
             <geometry>
-                <cylinder length="0.07" radius="0.06" />
-            </geometry>
-        </collision>
-        <xacro:inertial_cylinder mass="0.2" length="0.07" radius="0.06">
+                <cylinder length="0.075" radius="0.07" />
+            </geometry>
+        </collision>
+        <xacro:inertial_cylinder mass="0.2" length="0.07" radius="0.07">
             <origin xyz="0 0 0" rpy="0 0 0"/>
         </xacro:inertial_cylinder>
@@ -209,13 +298,13 @@
     <gazebo reference="rear_back_left_wheel">
         <material>Gazebo/Gray</material>
-        <mu1 value="0.3"/>
-        <mu2 value="0.3"/>
+        <mu1 value="0.5"/>
+        <mu2 value="0.5"/>
     </gazebo>
     <!-- ================================================== REAR BACK RIGHT WHEEL joint, link ================================================== -->
-    <joint name="rear_back_right_wheel_joint" type="fixed">
+    <joint name="rear_back_right_wheel_joint" type="continuous">
         <parent link="base_link"/>
         <child link="rear_back_right_wheel"/>
-        <origin xyz="-0.26 -0.225 0.01" rpy="${pi/2} 0 0"/>
-        <!--axis xyz="0 0 -1"/-->
+        <origin xyz="-0.26 -0.225 0" rpy="${pi/2} 0 0"/>
+        <axis xyz="0 0 -1"/>
     </joint>
     <!-- ================================================== -->
@@ -223,5 +312,5 @@
         <visual>
             <geometry>
-                <cylinder length="0.07" radius="0.06" />
+                <cylinder length="0.075" radius="0.07" />
             </geometry>
             <material name="gray"/>
@@ -229,8 +318,8 @@
         <collision>
             <geometry>
-                <cylinder length="0.07" radius="0.06" />
-            </geometry>
-        </collision>
-        <xacro:inertial_cylinder mass="0.2" length="0.07" radius="0.06">
+                <cylinder length="0.075" radius="0.07" />
+            </geometry>
+        </collision>
+        <xacro:inertial_cylinder mass="0.2" length="0.075" radius="0.07">
             <origin xyz="0 0 0" rpy="0 0 0"/>
         </xacro:inertial_cylinder>
@@ -238,6 +327,6 @@
     <gazebo reference="rear_back_right_wheel">
         <material>Gazebo/Gray</material>
-        <mu1 value="0.3"/>
-        <mu2 value="0.3"/>
+        <mu1 value="0.5"/>
+        <mu2 value="0.5"/>
     </gazebo>
 </robot>
