Commit message: add first gripper

File: src/articubot_one/description/gazebo_control.xacro (robot description, xacro)
@@ -19,5 +19,4 @@
             <odometry_frame>odom</odometry_frame>
             <robot_base_frame>base_link</robot_base_frame>
-            <command_topic>diff_cont/cmd_vel_unstamped</command_topic>  <!-- Match twist_mux -->
             <publish_odom>true</publish_odom>
             <publish_odom_tf>true</publish_odom_tf>
@@ -36,5 +35,4 @@
             <odometry_frame>odom</odometry_frame>
             <robot_base_frame>base_link</robot_base_frame>
-            <command_topic>diff_cont/cmd_vel_unstamped</command_topic>  <!-- Match twist_mux -->
             <publish_odom>true</publish_odom>
             <publish_odom_tf>true</publish_odom_tf>

File: src/articubot_one/description/gripper.xacro (robot description, xacro)
@@ -1,17 +1,26 @@
 <?xml version="1.0"?>
 <robot xmlns:xacro="http://www.ros.org/wiki/xacro" >
-    <!-- Gripper Base -->
+    <!-- ================================== Vertical Movement Joint for Gripper ================================== -->
+    <joint name="gripper_vertical_joint" type="prismatic">
+        <parent link="chassis"/>
+        <child link="gripper_base"/>
+        <origin xyz="0.25 0 0" rpy="0 0 1.57"/>
+        <axis xyz="0 0 1"/>
+        <limit effort="80" lower="0" upper="0.13" velocity="0.1"/>
+        <dynamics damping="50.0" friction="1.0"/>
+    </joint>
+    <!-- ================================== Gripper Base joint, link ================================== -->
     <link name="gripper_base">
         <visual>
             <origin xyz="0 0 0" rpy="0 0 0"/>
             <geometry>
-                <box size="0.35 0.05 0.05"/>
+                <box size="0.35 0.05 0.06"/>
             </geometry>
-            <material name="gray"/>
+            <material name="black"/>
         </visual>
         <collision>
             <origin xyz="0 0 0" rpy="0 0 0"/>
             <geometry>
-                <box size="0.35 0.05 0.05"/>
+                <box size="0.35 0.05 0.06"/>
             </geometry>
             <surface>
@@ -34,9 +43,18 @@
             </surface>
         </collision>
-        <xacro:inertial_box mass="0.5" x="0.35" y="0.05" z="0.05" >
+        <xacro:inertial_box mass="0.2" x="0.35" y="0.05" z="0.06" >
             <origin xyz="0 0 0" rpy="0 0 0"/>
         </xacro:inertial_box>
     </link>
-    <!-- Gripper Finger Left -->
+    <!-- ================================== Gripper Finger Left Joint ================================== -->
+    <joint name="gripper_finger_left_joint" type="prismatic">
+        <parent link="gripper_base"/>
+        <child link="gripper_finger_left"/>
+        <origin xyz="-0.075 0 0" rpy="0 0 0"/>
+        <axis xyz="1 0 0"/>
+        <limit effort="100" lower="0" upper="0.1" velocity="0.1"/>
+        <dynamics damping="20.0" friction="1.0"/>
+    </joint>
+    <!-- ================================== Gripper Finger Left link ================================== -->
     <link name="gripper_finger_left">
         <visual>
@@ -45,10 +63,10 @@
                 <box size="0.0225 0.2 0.05"/>
             </geometry>
-            <material name="orange"/>
+            <material name="blue"/>
         </visual>
         <collision>
             <origin xyz="-0.075 -0.1 0" rpy="0 0 0"/>
             <geometry>
-                <box size="0.0225 0.2 0.1"/>
+                <box size="0.0225 0.2 0.05"/>
             </geometry>
             <surface>
@@ -71,9 +89,18 @@
             </surface>
         </collision>
-        <xacro:inertial_box mass="0.3" x="0.0225" y="0.2" z="0.05" >
+        <xacro:inertial_box mass="0.1" x="0.0225" y="0.2" z="0.05" >
             <origin xyz="-0.075 -0.1 0" rpy="0 0 0"/>
         </xacro:inertial_box>
     </link>
-    <!-- Gripper Finger Right -->
+    <!-- ================================== Gripper Finger Right Joint ================================== -->
+    <joint name="gripper_finger_right_joint" type="prismatic">
+        <parent link="gripper_base"/>
+        <child link="gripper_finger_right"/>
+        <origin xyz="0.075 0 0" rpy="0 0 0"/>
+        <axis xyz="1 0 0"/>
+        <limit effort="100" lower="-0.1" upper="0" velocity="0.1"/>
+        <dynamics damping="20.0" friction="1.0"/>
+    </joint>
+    <!-- ================================== Gripper Finger Right link ================================== -->
     <link name="gripper_finger_right">
         <visual>
@@ -82,10 +109,10 @@
                 <box size="0.0225 0.2 0.05"/>
             </geometry>
-            <material name="orange"/>
+            <material name="blue"/>
         </visual>
         <collision>
             <origin xyz="0.075 -0.10 0" rpy="0 0 0"/>
             <geometry>
-                <box size="0.0225 0.2 0.1"/>
+                <box size="0.0225 0.2 0.05"/>
             </geometry>
             <surface>
@@ -108,37 +135,11 @@
             </surface>
         </collision>
-        <xacro:inertial_box mass="0.3" x="0.0225" y="0.2" z="0.05" >
-            <origin xyz="0.075 -0.10 0" rpy="0 0 0"/>
+        <xacro:inertial_box mass="0.1" x="0.0225" y="0.2" z="0.05" >
+            <origin xyz="0.075 -0.1 0" rpy="0 0 0"/>
         </xacro:inertial_box>
     </link>
-    <!-- Vertical Movement Joint for Gripper -->
-    <joint name="gripper_vertical_joint" type="prismatic">
-        <parent link="chassis"/>
-        <child link="gripper_base"/>
-        <origin xyz="0.25 0 0" rpy="0 0 1.57"/>
-        <axis xyz="0 0 1"/>
-        <limit effort="80" lower="0" upper="0.13" velocity="0.1"/>
-        <dynamics damping="50.0" friction="1.0"/>
-    </joint>
-    <!-- Gripper Finger Joints -->
-    <joint name="gripper_finger_left_joint" type="prismatic">
-        <parent link="gripper_base"/>
-        <child link="gripper_finger_left"/>
-        <origin xyz="-0.075 0 0" rpy="0 0 0"/>
-        <axis xyz="1 0 0"/>
-        <limit effort="100" lower="0" upper="0.1" velocity="0.1"/>
-        <dynamics damping="20.0" friction="1.0"/>
-    </joint>
-    <joint name="gripper_finger_right_joint" type="prismatic">
-        <parent link="gripper_base"/>
-        <child link="gripper_finger_right"/>
-        <origin xyz="0.075 0 0" rpy="0 0 0"/>
-        <axis xyz="1 0 0"/>
-        <limit effort="100" lower="-0.1" upper="0" velocity="0.1"/>
-        <dynamics damping="20.0" friction="1.0"/>
-    </joint>
-    <!-- Gazebo Simulation for Gripper -->
+    <!-- ================================== Gazebo Simulation for Gripper  ================================== -->
     <gazebo reference="gripper_base">
-        <material>Gazebo/Gray</material>
+        <material>Gazebo/Black</material>
         <gravity>true</gravity>
         <ode>
@@ -148,5 +149,5 @@
     </gazebo>
     <gazebo reference="gripper_finger_left">
-        <material>Gazebo/Orange</material>
+        <material>Gazebo/Blue</material>
         <gravity>true</gravity>
         <ode>
@@ -160,5 +161,5 @@
     </gazebo>
     <gazebo reference="gripper_finger_right">
-        <material>Gazebo/Orange</material>
+        <material>Gazebo/Blue</material>
         <gravity>true</gravity>
         <ode>

File: src/articubot_one/description/robot.urdf.xacro (robot description, xacro)
@@ -5,3 +5,17 @@
     <xacro:include filename="gazebo_control.xacro" />
     <xacro:include filename="lidar.xacro" />
+    <xacro:include filename="gripper.xacro" />
+    <xacro:include filename="gripper_vertical_tranmission.xacro" />
+    <xacro:include filename="gripper_finger_left_tranmission.xacro" />
+    <xacro:include filename="gripper_finger_right_tranmission.xacro" />
+    <xacro:include filename="robot_control.urdf.xacro"/>
+    <xacro:robot_controller/>
+    <ros2_control name="gripper_robot_gazebo_system" type="system">
+        <hardware>
+            <plugin>gazebo_ros2_control/GazeboSystem</plugin>
+        </hardware>
+        <xacro:gripper_vertical_tranmission/>
+        <xacro:gripper_finger_left_tranmission/>
+        <xacro:gripper_finger_right_tranmission/>
+    </ros2_control>
 </robot>

Commit message: add fiole

File: src/articubot_one/description/gazebo_control.xacro (robot description, xacro)
@@ -4,6 +4,4 @@
         <plugin name='diff_drive' filename='libgazebo_ros_diff_drive.so'>
             <!-- Wheel Information -->
-            <!-- <left_joint>front_left_wheel_joint</left_joint> -->
-            <!-- <right_joint>front_right_wheel_joint</right_joint> -->
             <num_wheel_pairs>2</num_wheel_pairs>
             <left_joint>back_left_wheel_joint</left_joint>
@@ -11,9 +9,9 @@
             <left_joint>front_left_wheel_joint</left_joint>
             <right_joint>front_right_wheel_joint</right_joint>
-            <wheel_separation>0.45</wheel_separation>  <!-- Distance between wheels (update if needed) -->
-            <wheel_diameter>0.14</wheel_diameter>        <!-- Diameter of the wheels (update if needed) -->
+            <wheel_separation>0.45</wheel_separation>
+            <wheel_diameter>0.14</wheel_diameter>
             <!-- Limits -->
             <max_wheel_torque>300</max_wheel_torque>
-            <max_wheel_acceleration>15.0</max_wheel_acceleration>
+            <max_wheel_acceleration>20.0</max_wheel_acceleration>
             <!-- Output -->
             <odometry_frame>odom</odometry_frame>
@@ -31,5 +29,5 @@
             <!-- Limits -->
             <max_wheel_torque>300</max_wheel_torque>
-            <max_wheel_acceleration>15.0</max_wheel_acceleration>
+            <max_wheel_acceleration>20.0</max_wheel_acceleration>
             <!-- Output -->
             <odometry_frame>odom</odometry_frame>

File: src/articubot_one/description/robot.urdf.xacro (robot description, xacro)
@@ -10,4 +10,5 @@
     <xacro:include filename="gripper_finger_right_tranmission.xacro" />
     <xacro:include filename="robot_control.urdf.xacro"/>
+    <!---
     <xacro:robot_controller/>
     <ros2_control name="gripper_robot_gazebo_system" type="system">
@@ -18,4 +19,4 @@
         <xacro:gripper_finger_left_tranmission/>
         <xacro:gripper_finger_right_tranmission/>
-    </ros2_control>
+    </ros2_control> -->
 </robot>

File: src/articubot_one/description/robot_core.xacro (robot description, xacro)
@@ -330,3 +330,24 @@
         <mu2 value="0.5"/>
     </gazebo>
+<!--
+<xacro:macro name="wheel_transmission" params="joint_name">
+  <transmission name="${joint_name}_trans">
+    <type>transmission_interface/SimpleTransmission</type>
+    <joint name="${joint_name}">
+      <hardware_interface>hardware_interface/VelocityJointInterface</hardware_interface>
+    </joint>
+    <actuator name="${joint_name}_actuator">
+      <hardware_interface>hardware_interface/VelocityJointInterface</hardware_interface>
+      <mechanical_reduction>1.0</mechanical_reduction>
+    </actuator>
+  </transmission>
+</xacro:macro>
+-->
+<!-- Call for each wheel joint
+<xacro:wheel_transmission joint_name="front_left_wheel_joint"/>
+<xacro:wheel_transmission joint_name="front_right_wheel_joint"/>
+<xacro:wheel_transmission joint_name="back_left_wheel_joint"/>
+<xacro:wheel_transmission joint_name="back_right_wheel_joint"/>
+<xacro:wheel_transmission joint_name="rear_back_left_wheel_joint"/>
+<xacro:wheel_transmission joint_name="rear_back_right_wheel_joint"/>  -->
 </robot>
