Commit message: add file2

File: src/articubot_one/description/robot_core.xacro (robot description, xacro)
@@ -46,5 +46,5 @@
     <link name="chassis">
         <visual>
-            <origin xyz="0 0 0.075" rpy="0 0 0"/>
+            <origin xyz="0 0 0.1" rpy="0 0 0"/>
             <geometry>
                 <box size="0.7 0.5 0.15"/>
@@ -58,5 +58,5 @@
             </geometry>
         </collision>
-        <xacro:inertial_box mass="0.5" x="0.7" y="0.5" z="0.15">
+        <xacro:inertial_box mass="0.8" x="0.7" y="0.5" z="0.15">
             <origin xyz="0 0 0.075" rpy="0 0 0"/>
         </xacro:inertial_box>
@@ -64,6 +64,6 @@
     <gazebo reference="chassis">
         <material>Gazebo/White</material>
-        <mu1 value="0.3"/>
-        <mu2 value="0.3"/>
+        <mu1 value="0.5"/>
+        <mu2 value="0.5"/>
     </gazebo>
     <!-- ==================================================  FRONT LEFT WHEEL joint, link ================================================== -->
@@ -71,5 +71,5 @@
         <parent link="base_link"/>
         <child link="front_left_wheel"/>
-        <origin xyz="0.17 0.27 0" rpy="-${pi/2} 0 0"/>
+        <origin xyz="0.17 0.225 0" rpy="-${pi/2} 0 0"/>
         <axis xyz="0 0 1"/>
     </joint>
@@ -78,5 +78,5 @@
         <visual>
             <geometry>
-                <cylinder length="0.04" radius="0.05" />
+                <cylinder length="0.07" radius="0.07" />
             </geometry>
             <material name="blue"/>
@@ -84,8 +84,8 @@
         <collision>
             <geometry>
-                <cylinder length="0.04" radius="0.05" />
+                <cylinder length="0.07" radius="0.05" />
             </geometry>
         </collision>
-        <xacro:inertial_cylinder mass="0.1" length="0.04" radius="0.05">
+        <xacro:inertial_cylinder mass="0.2" length="0.07" radius="0.07">
             <origin xyz="0 0 0" rpy="0 0 0"/>
         </xacro:inertial_cylinder>
@@ -93,6 +93,6 @@
     <gazebo reference="front_left_wheel">
         <material>Gazebo/Blue</material>
-        <mu1 value="0.3"/>
-        <mu2 value="0.3"/>
+        <mu1 value="0.5"/>
+        <mu2 value="0.5"/>
     </gazebo>
     <!-- ==================================================  FRONT RIGHT WHEEL joint, link ================================================== -->
@@ -100,5 +100,5 @@
         <parent link="base_link"/>
         <child link="front_right_wheel"/>
-        <origin xyz="0.17 -0.27 0" rpy="${pi/2} 0 0"/>
+        <origin xyz="0.17 -0.225 0" rpy="${pi/2} 0 0"/>
         <axis xyz="0 0 -1"/>
     </joint>
@@ -107,5 +107,5 @@
         <visual>
             <geometry>
-                <cylinder length="0.04" radius="0.05" />
+                <cylinder length="0.07" radius="0.07" />
             </geometry>
             <material name="blue"/>
@@ -113,8 +113,8 @@
         <collision>
             <geometry>
-                <cylinder length="0.04" radius="0.05" />
+                <cylinder length="0.07" radius="0.07" />
             </geometry>
         </collision>
-        <xacro:inertial_cylinder mass="0.1" length="0.04" radius="0.05">
+        <xacro:inertial_cylinder mass="0.2" length="0.07" radius="0.07">
             <origin xyz="0 0 0" rpy="0 0 0"/>
         </xacro:inertial_cylinder>
@@ -122,6 +122,6 @@
     <gazebo reference="front_right_wheel">
         <material>Gazebo/Blue</material>
-        <mu1 value="0.3"/>
-        <mu2 value="0.3"/>
+        <mu1 value="0.5"/>
+        <mu2 value="0.5"/>
     </gazebo>
     <!-- ==================================================  BACK LEFT WHEEL joint, link ================================================== -->
@@ -129,5 +129,5 @@
         <parent link="base_link"/>
         <child link="back_left_wheel"/>
-        <origin xyz="-0.1 0.27 0" rpy="-${pi/2} 0 0"/>
+        <origin xyz="-0.1 0.225 0" rpy="-${pi/2} 0 0"/>
         <axis xyz="0 0 1"/>
     </joint>
@@ -136,5 +136,5 @@
         <visual>
             <geometry>
-                <cylinder length="0.04" radius="0.05" />
+                <cylinder length="0.07" radius="0.07" />
             </geometry>
             <material name="gray"/>
@@ -142,8 +142,8 @@
         <collision>
             <geometry>
-                <cylinder length="0.04" radius="0.05" />
+                <cylinder length="0.07" radius="0.07" />
             </geometry>
         </collision>
-        <xacro:inertial_cylinder mass="0.1" length="0.04" radius="0.05">
+        <xacro:inertial_cylinder mass="0.2" length="0.07" radius="0.07">
             <origin xyz="0 0 0" rpy="0 0 0"/>
         </xacro:inertial_cylinder>
@@ -151,6 +151,6 @@
     <gazebo reference="back_left_wheel">
         <material>Gazebo/Gray</material>
-        <mu1 value="0.3"/>
-        <mu2 value="0.3"/>
+        <mu1 value="0.5"/>
+        <mu2 value="0.5"/>
     </gazebo>
     <!-- ================================================== BACK RIGHT WHEEL joint, link ================================================== -->
@@ -158,5 +158,5 @@
         <parent link="base_link"/>
         <child link="back_right_wheel"/>
-        <origin xyz="-0.1 -0.27 0" rpy="${pi/2} 0 0"/>
+        <origin xyz="-0.1 -0.225 0" rpy="${pi/2} 0 0"/>
         <axis xyz="0 0 -1"/>
     </joint>
@@ -165,5 +165,5 @@
         <visual>
             <geometry>
-                <cylinder length="0.04" radius="0.05" />
+                <cylinder length="0.07" radius="0.07" />
             </geometry>
             <material name="gray"/>
@@ -171,8 +171,8 @@
         <collision>
             <geometry>
-                <cylinder length="0.04" radius="0.05" />
+                <cylinder length="0.07" radius="0.07" />
             </geometry>
         </collision>
-        <xacro:inertial_cylinder mass="0.1" length="0.04" radius="0.05">
+        <xacro:inertial_cylinder mass="0.2" length="0.07" radius="0.07">
             <origin xyz="0 0 0" rpy="0 0 0"/>
         </xacro:inertial_cylinder>
@@ -180,6 +180,6 @@
     <gazebo reference="back_right_wheel">
         <material>Gazebo/Gray</material>
-        <mu1 value="0.3"/>
-        <mu2 value="0.3"/>
+        <mu1 value="0.5"/>
+        <mu2 value="0.5"/>
     </gazebo>
 </robot>

Commit message: fix

File: src/articubot_one/description/robot_core.xacro (robot description, xacro)
@@ -74,5 +74,5 @@
         <parent link="chassis"/>
         <child link="left_bumper"/>
-        <origin xyz="0.247 0.2 0.09" rpy="0 0 0"/>  <!-- Front edge of chassis -->
+        <origin xyz="0.247 0.2 0.09" rpy="0 0 0"/>
     </joint>
     <!-- ================================================== -->
@@ -80,5 +80,5 @@
         <visual>
             <geometry>
-                <cylinder length="0.12" radius="0.05"/>  <!-- Half chassis height -->
+                <cylinder length="0.12" radius="0.05"/>
             </geometry>
             <material name="white"/>
@@ -95,5 +95,5 @@
     <gazebo reference="left_bumper">
         <material>Gazebo/White</material>
-        <mu1 value="0.3"/>  <!-- Smoother sliding -->
+        <mu1 value="0.3"/>
         <mu2 value="0.3"/>
     </gazebo>
@@ -102,5 +102,5 @@
         <parent link="chassis"/>
         <child link="right_bumper"/>
-        <origin xyz="0.247 -0.2 0.09" rpy="0 0 0"/>  <!-- Rear edge of chassis -->
+        <origin xyz="0.247 -0.2 0.09" rpy="0 0 0"/>
     </joint>
     <!-- ================================================== -->
