Commit message: fix2

File: src/articubot_one/description/gripper.xacro (robot description, xacro)
@@ -43,5 +43,5 @@
             </surface>
         </collision>
-        <xacro:inertial_box mass="0.2" x="0.35" y="0.05" z="0.06" >
+        <xacro:inertial_box mass="0.1" x="0.35" y="0.05" z="0.06" >
             <origin xyz="0 0 0" rpy="0 0 0"/>
         </xacro:inertial_box>
@@ -89,5 +89,5 @@
             </surface>
         </collision>
-        <xacro:inertial_box mass="0.1" x="0.0225" y="0.2" z="0.05" >
+        <xacro:inertial_box mass="0.05" x="0.0225" y="0.2" z="0.05" >
             <origin xyz="-0.075 -0.1 0" rpy="0 0 0"/>
         </xacro:inertial_box>
@@ -135,5 +135,5 @@
             </surface>
         </collision>
-        <xacro:inertial_box mass="0.1" x="0.0225" y="0.2" z="0.05" >
+        <xacro:inertial_box mass="0.05" x="0.0225" y="0.2" z="0.05" >
             <origin xyz="0.075 -0.1 0" rpy="0 0 0"/>
         </xacro:inertial_box>

File: src/articubot_one/description/gripper_tranmission.xacro (robot description, xacro)
@@ -1,23 +1,33 @@
 <?xml version="1.0"?>
-<robot xmlns:xacro="http://www.ros.org/wiki/xacro">
-    <xacro:macro name="gripper_transmission" params="">
-        <transmission name="gripper_trans">
-            <type>transmission_interface/SimpleTransmission</type>
-            <joint name="gripper_vertical_joint">
-                <command_interface name="position" />
-                <state_interface name="position" />
-                <state_interface name="velocity" />
-            </joint>
-            <joint name="gripper_finger_left_joint">
-                <command_interface name="position" />
-                <state_interface name="position" />
-                <state_interface name="velocity" />
-            </joint>
-            <joint name="gripper_finger_right_joint">
-                <command_interface name="position" />
-                <state_interface name="position" />
-                <state_interface name="velocity" />
-            </joint>
-        </transmission>
+<robot xmlns:xacro="http://ros.org/wiki/xacro">
+    <xacro:macro name="gripper_finger_left_tranmission" params="">
+        <joint name="gripper_finger_left_joint">
+            <command_interface name="velocity">
+                <param name="min">0</param>
+                <param name="max">0.1</param>
+            </command_interface>
+            <state_interface name="position" />
+            <state_interface name="velocity" />
+        </joint>
+    </xacro:macro>
+    <xacro:macro name="gripper_finger_right_tranmission" params="">
+        <joint name="gripper_finger_right_joint">
+            <command_interface name="velocity">
+                <param name="min">-0.1</param>
+                <param name="max">0</param>
+            </command_interface>
+            <state_interface name="position" />
+            <state_interface name="velocity" />
+        </joint>
+    </xacro:macro>
+    <xacro:macro name="gripper_vertical_tranmission" params="">
+        <joint name="gripper_vertical_joint">
+            <command_interface name="velocity">
+                <param name="min">0</param>
+                <param name="max">0.13</param>
+            </command_interface>
+            <state_interface name="position" />
+            <state_interface name="velocity" />
+        </joint>
     </xacro:macro>
 </robot>

File: src/articubot_one/description/robot.urdf.xacro (robot description, xacro)
@@ -6,9 +6,6 @@
     <xacro:include filename="lidar.xacro" />
     <xacro:include filename="gripper.xacro" />
-    <xacro:include filename="gripper_vertical_tranmission.xacro" />
-    <xacro:include filename="gripper_finger_left_tranmission.xacro" />
-    <xacro:include filename="gripper_finger_right_tranmission.xacro" />
-    <xacro:include filename="robot_control.urdf.xacro"/>
-    <!---
+    <xacro:include filename="gripper_tranmission.xacro" />
+    <xacro:include filename="gazebo_plugin.xacro"/>
     <xacro:robot_controller/>
     <ros2_control name="gripper_robot_gazebo_system" type="system">
@@ -19,4 +16,4 @@
         <xacro:gripper_finger_left_tranmission/>
         <xacro:gripper_finger_right_tranmission/>
-    </ros2_control> -->
+    </ros2_control>
 </robot>

Commit message: gripper can grab

File: src/articubot_one/description/gripper.xacro (robot description, xacro)
@@ -27,6 +27,6 @@
                 <friction>
                     <ode>
-                        <mu>2.0</mu>  <!-- Increase primary friction -->
-                        <mu2>2.0</mu2>  <!-- Increase secondary friction -->
+                        <mu>3.0</mu>  <!-- Increase primary friction -->
+                        <mu2>3.0</mu2>  <!-- Increase secondary friction -->
                     </ode>
                 </friction>
@@ -61,5 +61,5 @@
             <origin xyz="-0.075 -0.1 0" rpy="0 0 0"/>
             <geometry>
-                <box size="0.0225 0.2 0.05"/>
+                <box size="0.0225 0.2 0.06"/>
             </geometry>
             <material name="blue"/>
@@ -68,11 +68,11 @@
             <origin xyz="-0.075 -0.1 0" rpy="0 0 0"/>
             <geometry>
-                <box size="0.0225 0.2 0.05"/>
+                <box size="0.0225 0.2 0.06"/>
             </geometry>
             <surface>
                 <friction>
                     <ode>
-                        <mu>2.0</mu>  <!-- Increase primary friction -->
-                        <mu2>2.0</mu2>  <!-- Increase secondary friction -->
+                        <mu>3.0</mu>  <!-- Increase primary friction -->
+                        <mu2>3.0</mu2>  <!-- Increase secondary friction -->
                     </ode>
                 </friction>
@@ -89,5 +89,5 @@
             </surface>
         </collision>
-        <xacro:inertial_box mass="0.05" x="0.0225" y="0.2" z="0.05" >
+        <xacro:inertial_box mass="0.1" x="0.0225" y="0.2" z="0.06" >
             <origin xyz="-0.075 -0.1 0" rpy="0 0 0"/>
         </xacro:inertial_box>
@@ -107,5 +107,5 @@
             <origin xyz="0.075 -0.10 0" rpy="0 0 0"/>
             <geometry>
-                <box size="0.0225 0.2 0.05"/>
+                <box size="0.0225 0.2 0.06"/>
             </geometry>
             <material name="blue"/>
@@ -114,11 +114,11 @@
             <origin xyz="0.075 -0.10 0" rpy="0 0 0"/>
             <geometry>
-                <box size="0.0225 0.2 0.05"/>
+                <box size="0.0225 0.2 0.06"/>
             </geometry>
             <surface>
                 <friction>
                     <ode>
-                        <mu>2.0</mu>  <!-- Increase primary friction -->
-                        <mu2>2.0</mu2>  <!-- Increase secondary friction -->
+                        <mu>3.0</mu>  <!-- Increase primary friction -->
+                        <mu2>3.0</mu2>  <!-- Increase secondary friction -->
                     </ode>
                 </friction>
@@ -135,5 +135,5 @@
             </surface>
         </collision>
-        <xacro:inertial_box mass="0.05" x="0.0225" y="0.2" z="0.05" >
+        <xacro:inertial_box mass="0.1" x="0.0225" y="0.2" z="0.06" >
             <origin xyz="0.075 -0.1 0" rpy="0 0 0"/>
         </xacro:inertial_box>

File: src/articubot_one/description/robot_core.xacro (robot description, xacro)
@@ -61,5 +61,5 @@
             </geometry>
         </collision>
-        <xacro:inertial_box mass="0.4" x="0.6" y="0.5" z="0.15">
+        <xacro:inertial_box mass="150.0" x="0.6" y="0.5" z="0.15">
             <origin xyz="0 0 0.075" rpy="0 0 0"/>
         </xacro:inertial_box>
@@ -89,5 +89,5 @@
             </geometry>
         </collision>
-        <xacro:inertial_cylinder mass="0.1" length="0.12" radius="0.05">
+        <xacro:inertial_cylinder mass="10.0" length="0.12" radius="0.05">
             <origin xyz="0 0 0" rpy="0 0 0"/>
         </xacro:inertial_cylinder>
@@ -117,5 +117,5 @@
             </geometry>
         </collision>
-        <xacro:inertial_cylinder mass="0.1" length="0.12" radius="0.05">
+        <xacro:inertial_cylinder mass="10.0" length="0.12" radius="0.05">
             <origin xyz="0 0 0" rpy="0 0 0"/>
         </xacro:inertial_cylinder>
@@ -147,5 +147,5 @@
             </geometry>
         </collision>
-        <xacro:inertial_box mass="0.1" x="0.05" y="0.4" z="0.1">
+        <xacro:inertial_box mass="10.0" x="0.05" y="0.4" z="0.1">
             <origin xyz="0 0 0.05" rpy="0 0 0"/>
         </xacro:inertial_box>
@@ -176,5 +176,5 @@
             </geometry>
         </collision>
-        <xacro:inertial_cylinder mass="0.2" length="0.075" radius="0.07">
+        <xacro:inertial_cylinder mass="20.0" length="0.075" radius="0.07">
             <origin xyz="0 0 0" rpy="0 0 0"/>
         </xacro:inertial_cylinder>
@@ -205,5 +205,5 @@
             </geometry>
         </collision>
-        <xacro:inertial_cylinder mass="0.2" length="0.075" radius="0.07">
+        <xacro:inertial_cylinder mass="20.0" length="0.075" radius="0.07">
             <origin xyz="0 0 0" rpy="0 0 0"/>
         </xacro:inertial_cylinder>
@@ -234,5 +234,5 @@
             </geometry>
         </collision>
-        <xacro:inertial_cylinder mass="0.2" length="0.075" radius="0.07">
+        <xacro:inertial_cylinder mass="20.0" length="0.075" radius="0.07">
             <origin xyz="0 0 0" rpy="0 0 0"/>
         </xacro:inertial_cylinder>
@@ -263,5 +263,5 @@
             </geometry>
         </collision>
-        <xacro:inertial_cylinder mass="0.2" length="0.075" radius="0.07">
+        <xacro:inertial_cylinder mass="20.0" length="0.075" radius="0.07">
             <origin xyz="0 0 0" rpy="0 0 0"/>
         </xacro:inertial_cylinder>
@@ -292,5 +292,5 @@
             </geometry>
         </collision>
-        <xacro:inertial_cylinder mass="0.2" length="0.07" radius="0.07">
+        <xacro:inertial_cylinder mass="20.0" length="0.07" radius="0.07">
             <origin xyz="0 0 0" rpy="0 0 0"/>
         </xacro:inertial_cylinder>
@@ -321,5 +321,5 @@
             </geometry>
         </collision>
-        <xacro:inertial_cylinder mass="0.2" length="0.075" radius="0.07">
+        <xacro:inertial_cylinder mass="20.0" length="0.075" radius="0.07">
             <origin xyz="0 0 0" rpy="0 0 0"/>
         </xacro:inertial_cylinder>

Commit message: fix friction

File: src/articubot_one/description/gripper.xacro (robot description, xacro)
@@ -15,5 +15,5 @@
             <origin xyz="0 0 0" rpy="0 0 0"/>
             <geometry>
-                <box size="0.35 0.05 0.06"/>
+                <box size="0.35 0.05 0.07"/>
             </geometry>
             <material name="black"/>
@@ -22,5 +22,5 @@
             <origin xyz="0 0 0" rpy="0 0 0"/>
             <geometry>
-                <box size="0.35 0.05 0.06"/>
+                <box size="0.35 0.05 0.07"/>
             </geometry>
             <surface>
@@ -43,5 +43,5 @@
             </surface>
         </collision>
-        <xacro:inertial_box mass="0.1" x="0.35" y="0.05" z="0.06" >
+        <xacro:inertial_box mass="0.1" x="0.35" y="0.05" z="0.07" >
             <origin xyz="0 0 0" rpy="0 0 0"/>
         </xacro:inertial_box>
@@ -61,5 +61,5 @@
             <origin xyz="-0.075 -0.1 0" rpy="0 0 0"/>
             <geometry>
-                <box size="0.0225 0.2 0.06"/>
+                <box size="0.0225 0.2 0.07"/>
             </geometry>
             <material name="blue"/>
@@ -68,11 +68,11 @@
             <origin xyz="-0.075 -0.1 0" rpy="0 0 0"/>
             <geometry>
-                <box size="0.0225 0.2 0.06"/>
+                <box size="0.0225 0.2 0.07"/>
             </geometry>
             <surface>
                 <friction>
                     <ode>
-                        <mu>5.0</mu>  <!-- Increase primary friction -->
-                        <mu2>5.0</mu2>  <!-- Increase secondary friction -->
+                        <mu>7.0</mu>  <!-- Increase primary friction -->
+                        <mu2>7.0</mu2>  <!-- Increase secondary friction -->
                     </ode>
                 </friction>
@@ -89,5 +89,5 @@
             </surface>
         </collision>
-        <xacro:inertial_box mass="0.1" x="0.0225" y="0.2" z="0.06" >
+        <xacro:inertial_box mass="0.1" x="0.0225" y="0.2" z="0.07" >
             <origin xyz="-0.075 -0.1 0" rpy="0 0 0"/>
         </xacro:inertial_box>
@@ -107,5 +107,5 @@
             <origin xyz="0.075 -0.10 0" rpy="0 0 0"/>
             <geometry>
-                <box size="0.0225 0.2 0.06"/>
+                <box size="0.0225 0.2 0.07"/>
             </geometry>
             <material name="blue"/>
@@ -114,11 +114,11 @@
             <origin xyz="0.075 -0.10 0" rpy="0 0 0"/>
             <geometry>
-                <box size="0.0225 0.2 0.06"/>
+                <box size="0.0225 0.2 0.07"/>
             </geometry>
             <surface>
                 <friction>
                     <ode>
-                        <mu>5.0</mu>  <!-- Increase primary friction -->
-                        <mu2>5.0</mu2>  <!-- Increase secondary friction -->
+                        <mu>7.0</mu>  <!-- Increase primary friction -->
+                        <mu2>7.0</mu2>  <!-- Increase secondary friction -->
                     </ode>
                 </friction>
@@ -135,5 +135,5 @@
             </surface>
         </collision>
-        <xacro:inertial_box mass="0.1" x="0.0225" y="0.2" z="0.06" >
+        <xacro:inertial_box mass="0.1" x="0.0225" y="0.2" z="0.07" >
             <origin xyz="0.075 -0.1 0" rpy="0 0 0"/>
         </xacro:inertial_box>
