Commit message: finish presentation

File: src/articubot_one/description/gripper_core.xacro (robot description, xacro)
@@ -7,6 +7,6 @@
         <origin xyz="0.25 0 0" rpy="0 0 1.57"/>
         <axis xyz="0 0 1"/>
-        <limit effort="80" lower="0" upper="0.13" velocity="0.1"/>
-        <dynamics damping="50.0" friction="1.0"/>
+        <limit effort="80" lower="0" upper="0.13" velocity="0.3"/>
+        <dynamics damping="50.0" friction="2.0"/>
     </joint>
     <!-- ================================== Gripper Base joint, link ================================== -->
@@ -15,5 +15,5 @@
             <origin xyz="0 0 0" rpy="0 0 0"/>
             <geometry>
-                <box size="0.35 0.05 0.07"/>
+                <box size="0.35 0.05 0.1"/>
             </geometry>
             <material name="black"/>
@@ -22,5 +22,5 @@
             <origin xyz="0 0 0" rpy="0 0 0"/>
             <geometry>
-                <box size="0.35 0.05 0.07"/>
+                <box size="0.35 0.05 0.1"/>
             </geometry>
             <surface>
@@ -43,5 +43,5 @@
             </surface>
         </collision>
-        <xacro:inertial_box mass="0.1" x="0.35" y="0.05" z="0.07" >
+        <xacro:inertial_box mass="0.1" x="0.35" y="0.05" z="0.1" >
             <origin xyz="0 0 0" rpy="0 0 0"/>
         </xacro:inertial_box>
@@ -51,8 +51,8 @@
         <parent link="gripper_base"/>
         <child link="gripper_finger_left"/>
-        <origin xyz="-0.075 0 0" rpy="0 0 0"/>
+        <origin xyz="-0.075 -0.02 0" rpy="0 0 0"/>
         <axis xyz="1 0 0"/>
-        <limit effort="100" lower="0" upper="0.1" velocity="0.1"/>
-        <dynamics damping="20.0" friction="1.0"/>
+        <limit effort="100" lower="0" upper="0.1" velocity="0.35"/>
+        <dynamics damping="20.0" friction="6.5"/>
     </joint>
     <!-- ================================== Gripper Finger Left link ================================== -->
@@ -61,18 +61,18 @@
             <origin xyz="-0.075 -0.1 0" rpy="0 0 0"/>
             <geometry>
-                <box size="0.0225 0.2 0.07"/>
+                <box size="0.03 0.2 0.1"/>
             </geometry>
             <material name="blue"/>
         </visual>
         <collision>
-            <origin xyz="-0.075 -0.1 0" rpy="0 0 0"/>
+            <origin xyz="-0.075 -0.075 0" rpy="0 0 0"/>
             <geometry>
-                <box size="0.0225 0.2 0.07"/>
+                <box size="0.03 0.2 0.1"/>
             </geometry>
             <surface>
                 <friction>
                     <ode>
-                        <mu>7.0</mu>  <!-- Increase primary friction -->
-                        <mu2>7.0</mu2>  <!-- Increase secondary friction -->
+                        <mu>10.0</mu>  <!-- Increase primary friction -->
+                        <mu2>10.0</mu2>  <!-- Increase secondary friction -->
                     </ode>
                 </friction>
@@ -89,5 +89,5 @@
             </surface>
         </collision>
-        <xacro:inertial_box mass="0.1" x="0.0225" y="0.2" z="0.07" >
+        <xacro:inertial_box mass="1" x="0.03" y="0.2" z="0.1" >
             <origin xyz="-0.075 -0.1 0" rpy="0 0 0"/>
         </xacro:inertial_box>
@@ -97,28 +97,28 @@
         <parent link="gripper_base"/>
         <child link="gripper_finger_right"/>
-        <origin xyz="0.075 0 0" rpy="0 0 0"/>
+        <origin xyz="0.075 -0.02 0" rpy="0 0 0"/>
         <axis xyz="1 0 0"/>
-        <limit effort="100" lower="-0.1" upper="0" velocity="0.1"/>
-        <dynamics damping="20.0" friction="1.0"/>
+        <limit effort="100" lower="-0.1" upper="0" velocity="0.35"/>
+        <dynamics damping="20.0" friction="6.5"/>
     </joint>
     <!-- ================================== Gripper Finger Right link ================================== -->
     <link name="gripper_finger_right">
         <visual>
-            <origin xyz="0.075 -0.10 0" rpy="0 0 0"/>
+            <origin xyz="0.075 -0.1 0" rpy="0 0 0"/>
             <geometry>
-                <box size="0.0225 0.2 0.07"/>
+                <box size="0.035 0.2 0.1"/>
             </geometry>
             <material name="blue"/>
         </visual>
         <collision>
-            <origin xyz="0.075 -0.10 0" rpy="0 0 0"/>
+            <origin xyz="0.075 -0.075 0" rpy="0 0 0"/>
             <geometry>
-                <box size="0.0225 0.2 0.07"/>
+                <box size="0.035 0.2 0.1"/>
             </geometry>
             <surface>
                 <friction>
                     <ode>
-                        <mu>7.0</mu>  <!-- Increase primary friction -->
-                        <mu2>7.0</mu2>  <!-- Increase secondary friction -->
+                        <mu>10.0</mu>  <!-- Increase primary friction -->
+                        <mu2>10.0</mu2>  <!-- Increase secondary friction -->
                     </ode>
                 </friction>
@@ -135,5 +135,5 @@
             </surface>
         </collision>
-        <xacro:inertial_box mass="0.1" x="0.0225" y="0.2" z="0.07" >
+        <xacro:inertial_box mass="1" x="0.035" y="0.2" z="0.1" >
             <origin xyz="0.075 -0.1 0" rpy="0 0 0"/>
         </xacro:inertial_box>

File: src/articubot_one/description/robot.urdf.xacro (robot description, xacro)
@@ -5,6 +5,6 @@
     <xacro:include filename="gazebo_control.xacro" />
     <xacro:include filename="lidar.xacro" />
-    <xacro:include filename="gripper.xacro" />
-    <xacro:include filename="gripper_tranmission.xacro" />
+    <xacro:include filename="gripper_core.xacro" />
+    <xacro:include filename="gripper_urdf.xacro" />
     <xacro:include filename="gazebo_plugin.xacro"/>
     <xacro:robot_controller/>
